File: SensorControlBoard/perepherals.kicad_sch (KiCad schematic)
At the start: 42 parts, among them J1 Micro_SD_Card, U10 ASMB-TTF0-0A20B, U11 ASMB-TTF0-0A20B, U12 AT24CS04-XHM, U13 OPT3002DNPR, U5 LP5018RSMR, U6 ASMB-TTF0-0A20B, U7 ASMB-TTF0-0A20B, U8 ASMB-TTF0-0A20B, U9 ASMB-TTF0-0A20B

Commit message: Initial Routing finished
Connections:
- net GPIO_2 is gone; now on net GPIO_6: R?.2, R?.2, U?.8 (~{ALERT})
- net GPIO_3 is gone; now on net GPIO_8: U5.30 (EN)
- net GPIO_4 is gone; now on net GPIO_7: D?.1 (K), R?.2, U?.5 (~{INT})
- net GPIO_6: no longer R2.1, R?.2, U13.5 (INT)
- net GPIO_7: no longer MT1.4 (INT1/INT)
- net GPIO_8: no longer MT1.9 (INT2)
- net GPIO_1 renamed GPIO_11
- net GPIO_5 renamed GPIO_9
- new net GPIO_12: R2.1, R?.2, U13.5 (INT)
- new net GPIO_13: MT1.9 (INT2)
- new net GPIO_14: MT1.4 (INT1/INT)
Changed lines of the file:
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@@
   (junction (at 154.178 206.502) (diameter 0) (color 0 0 0 0)
   )
+  (junction (at 103.886 57.15) (diameter 0) (color 0 0 0 0)
+  )
   (junction (at 56.642 199.136) (diameter 0) (color 0 0 0 0)
   )
@@
   )
   (junction (at 217.932 60.96) (diameter 0) (color 0 0 0 0)
-  )
-  (junction (at 103.886 57.15) (diameter 0) (color 0 0 0 0)
   )
   (junction (at 46.228 211.836) (diameter 0) (color 0 0 0 0)
@@
     (stroke (width 0) (type default))
   )
+  (wire (pts (xy 103.886 57.15) (xy 117.856 57.15))
+    (stroke (width 0) (type default))
+  )
   (wire (pts (xy 70.358 210.312) (xy 70.358 211.836))
     (stroke (width 0) (type default))
@@
     (stroke (width 0) (type default))
   )
-  (wire (pts (xy 117.856 57.15) (xy 103.886 57.15))
-    (stroke (width 0) (type default))
-  )
   (wire (pts (xy 46.228 227.33) (xy 46.228 229.108))
     (stroke (width 0) (type default))
@@
     (stroke (width 0) (type default))
   )
-  (wire (pts (xy 103.886 57.15) (xy 103.886 63.246))
-    (stroke (width 0) (type default))
-  )
   (wire (pts (xy 154.178 198.12) (xy 154.178 206.502))
     (stroke (width 0) (type default))
@@
   )
   (wire (pts (xy 166.37 206.502) (xy 166.37 210.566))
+    (stroke (width 0) (type default))
+  )
+  (wire (pts (xy 103.886 57.15) (xy 103.886 61.849))
     (stroke (width 0) (type default))
   )
@@
     (effects (font (size 1.27 1.27)) (justify left bottom))
   )
-  (global_label "GPIO_2" (shape bidirectional) (at 217.932 66.04 270) (fields_autoplaced)
+  (global_label "GPIO_6" (shape bidirectional) (at 217.932 66.04 270) (fields_autoplaced)
     (effects (font (size 1.27 1.27)) (justify right))
     (property "Intersheetrefs" "${INTERSHEET_REFS}" (at 217.932 76.7889 90)
@@
     )
   )
-  (global_label "GPIO_5" (shape bidirectional) (at 67.31 211.836 180) (fields_autoplaced)
+  (global_label "GPIO_9" (shape bidirectional) (at 67.31 211.836 180) (fields_autoplaced)
     (effects (font (size 1.27 1.27)) (justify right))
     (property "Intersheetrefs" "${INTERSHEET_REFS}" (at 56.5611 211.836 0)
@@
     )
   )
-  (global_label "GPIO_8" (shape bidirectional) (at 225.298 136.144 0) (fields_autoplaced)
+  (global_label "GPIO_13" (shape bidirectional) (at 225.298 136.144 0) (fields_autoplaced)
     (effects (font (size 1.27 1.27)) (justify left))
-    (property "Intersheetrefs" "${INTERSHEET_REFS}" (at 236.0469 136.144 0)
+    (property "Intersheetrefs" "${INTERSHEET_REFS}" (at 237.2564 136.144 0)
       (effects (font (size 1.27 1.27)) (justify left) hide)
     )
@@
     )
   )
-  (global_label "GPIO_7" (shape bidirectional) (at 225.298 133.604 0) (fields_autoplaced)
+  (global_label "GPIO_14" (shape bidirectional) (at 225.298 133.604 0) (fields_autoplaced)
     (effects (font (size 1.27 1.27)) (justify left))
-    (property "Intersheetrefs" "${INTERSHEET_REFS}" (at 236.0469 133.604 0)
+    (property "Intersheetrefs" "${INTERSHEET_REFS}" (at 237.2564 133.604 0)
       (effects (font (size 1.27 1.27)) (justify left) hide)
-    )
-  )
-  (global_label "GPIO_4" (shape bidirectional) (at 103.886 63.246 270) (fields_autoplaced)
-    (effects (font (size 1.27 1.27)) (justify right))
-    (property "Intersheetrefs" "${INTERSHEET_REFS}" (at 103.886 73.9949 90)
-      (effects (font (size 1.27 1.27)) (justify right) hide)
     )
   )
@@
     )
   )
-  (global_label "GPIO_6" (shape bidirectional) (at 232.156 225.044 270) (fields_autoplaced)
-    (effects (font (size 1.27 1.27)) (justify right))
-    (property "Intersheetrefs" "${INTERSHEET_REFS}" (at 232.156 235.7929 90)
+  (global_label "GPIO_7" (shape bidirectional) (at 103.886 61.849 270) (fields_autoplaced)
+    (effects (font (size 1.27 1.27)) (justify right))
+    (property "Intersheetrefs" "${INTERSHEET_REFS}" (at 103.886 72.5979 90)
+      (effects (font (size 1.27 1.27)) (justify right) hide)
+    )
+  )
+  (global_label "GPIO_12" (shape bidirectional) (at 232.156 225.044 270) (fields_autoplaced)
+    (effects (font (size 1.27 1.27)) (justify right))
+    (property "Intersheetrefs" "${INTERSHEET_REFS}" (at 232.156 237.0024 90)
       (effects (font (size 1.27 1.27)) (justify right) hide)
     )
@@
     )
   )
-  (global_label "GPIO_3" (shape bidirectional) (at 281.686 64.516 180) (fields_autoplaced)
+  (global_label "GPIO_8" (shape bidirectional) (at 281.686 64.516 180) (fields_autoplaced)
     (effects (font (size 1.27 1.27)) (justify right))
     (property "Intersheetrefs" "${INTERSHEET_REFS}" (at 270.9371 64.516 0)
@@
     )
   )
-  (global_label "GPIO_1" (shape bidirectional) (at 161.29 68.58 180) (fields_autoplaced)
-    (effects (font (size 1.27 1.27)) (justify right))
-    (property "Intersheetrefs" "${INTERSHEET_REFS}" (at 150.5411 68.58 0)
-      (effects (font (size 1.27 1.27)) (justify right) hide)
-    )
+  (global_label "GPIO_11" (shape bidirectional) (at 161.29 68.58 180) (fields_autoplaced)
+    (effects (font (size 1.27 1.27)) (justify right))
+    (property "Intersheetrefs" "${INTERSHEET_REFS}" (at 149.3316 68.58 0)
+      (effects (font (size 1.27 1.27)) (justify right) hide)
+    )

Commit message: A0 PCB Commit
Parts:
- C1: MP C0805C104K5RAC7210 -> C0603C104M4RAC7411
- C? (x8): MP C0805C105Z4VAC7800 -> C0603C105K4RACTU
- J1: MP 2508051217Y6 -> DM3D-SF
- U12: MP (none) -> AT24CS04-XHM
- U13: MP (none) -> OPT3002DNPR
- U14: renamed from MT1; MP (none) -> ICM-42670-P
- U?: MP (none) -> TMAG5170-Q1
- U?: MP (none) -> TMAG5273B1QDBVR
Changed lines of the file:
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@@
       (effects (font (size 1.27 1.27)) hide)
     )
-    (property "MP" "2508051217Y6" (at 98.044 216.916 0)
+    (property "MP" "DM3D-SF" (at 98.044 216.916 0)
       (effects (font (size 1.27 1.27)) hide)
     )
@@
       (effects (font (size 1.27 1.27)) hide)
     )
-    (property "MP" "C0805C105Z4VAC7800" (at 181.61 48.26 0)
+    (property "MP" "C0603C105K4RACTU" (at 181.61 48.26 0)
       (effects (font (size 1.27 1.27)) hide)
     )
@@
       (effects (font (size 1.27 1.27)) hide)
     )
-    (property "MP" "C0805C105Z4VAC7800" (at 148.082 211.582 0)
+    (property "MP" "C0603C105K4RACTU" (at 148.082 211.582 0)
       (effects (font (size 1.27 1.27)) hide)
     )
@@
       (effects (font (size 1.27 1.27)) hide)
     )
+    (property "MP" "AT24CS04-XHM" (at 80.01 143.256 0)
+      (effects (font (size 1.27 1.27)) hide)
+    )
     (pin "1")
     (pin "2")
@@
       (effects (font (size 1.27 1.27)) hide)
     )
-    (property "MP" "C0805C105Z4VAC7800" (at 303.784 135.128 0)
+    (property "MP" "C0603C105K4RACTU" (at 303.784 135.128 0)
       (effects (font (size 1.27 1.27)) hide)
     )
@@
       (effects (font (size 1.27 1.27)) hide)
     )
-    (property "MP" "C0805C104K5RAC7210" (at 216.916 117.348 0)
+    (property "MP" "C0603C104M4RAC7411" (at 216.916 117.348 0)
       (effects (font (size 1.27 1.27)) hide)
     )
@@
       (effects (font (size 1.27 1.27)) hide)
     )
+    (property "MP" "TMAG5170-Q1" (at 197.358 68.58 0)
+      (effects (font (size 1.27 1.27)) hide)
+    )
     (pin "1")
     (pin "2")
@@
       (effects (font (size 1.27 1.27)) hide)
     )
-    (property "MP" "C0805C105Z4VAC7800" (at 42.164 219.202 0)
+    (property "MP" "C0603C105K4RACTU" (at 42.164 219.202 0)
       (effects (font (size 1.27 1.27)) hide)
     )
@@
       (effects (font (size 1.27 1.27)) hide)
     )
+    (property "MP" "TMAG5273B1QDBVR" (at 82.042 64.77 0)
+      (effects (font (size 1.27 1.27)) hide)
+    )
     (pin "1")
     (pin "2")
@@
       (effects (font (size 1.27 1.27)) hide)
     )
-    (property "MP" "C0805C105Z4VAC7800" (at 240.538 117.348 0)
+    (property "MP" "C0603C105K4RACTU" (at 240.538 117.348 0)
       (effects (font (size 1.27 1.27)) hide)
     )
@@
   (symbol (lib_id "ICM-42670-P:ICM-42670-P") (at 193.04 136.144 0) (unit 1)
     (in_bom yes) (on_board yes) (dnp no) (fields_autoplaced)
-    (property "Reference" "MT1" (at 193.04 118.11 0)
+    (property "Reference" "U14" (at 193.04 118.11 0)
       (effects (font (size 1.27 1.27)))
     )
@@
       (effects (font (size 1.27 1.27)) (justify bottom) hide)
     )
+    (property "MP" "ICM-42670-P" (at 193.04 136.144 0)
+      (effects (font (size 1.27 1.27)) hide)
+    )
     (pin "1")
     (pin "10")
@@
       (project "SensorControlBoard"
         (path "/8c0c4014-aa51-4bf6-8434-aa4d122163d4/08ebbf42-81e7-4a5c-bbac-f4d91ee3da15"
-          (reference "MT1") (unit 1)
+          (reference "U14") (unit 1)
         )
       )
@@
       (effects (font (size 1.27 1.27) italic) hide)
     )
+    (property "MP" "OPT3002DNPR" (at 168.656 210.566 0)
+      (effects (font (size 1.27 1.27)) hide)
+    )
     (pin "1")
     (pin "2")
@@
       (effects (font (size 1.27 1.27)) hide)
     )
-    (property "MP" "C0805C105Z4VAC7800" (at 50.038 48.768 0)
+    (property "MP" "C0603C105K4RACTU" (at 50.038 48.768 0)
       (effects (font (size 1.27 1.27)) hide)
     )
@@
       (effects (font (size 1.27 1.27)) hide)
     )
-    (property "MP" "C0805C105Z4VAC7800" (at 49.276 134.366 0)
+    (property "MP" "C0603C105K4RACTU" (at 49.276 134.366 0)
       (effects (font (size 1.27 1.27)) hide)
     )
@@
       (effects (font (size 1.27 1.27)) hide)
     )
-    (property "MP" "C0805C104K5RAC7210" (at 230.378 116.84 0)
+    (property "MP" "C0603C104M4RAC7411" (at 230.378 116.84 0)
       (effects (font (size 1.27 1.27)) hide)
     )
@@
       (effects (font (size 1.27 1.27)) hide)
     )
-    (property "MP" "C0805C105Z4VAC7800" (at 281.686 55.626 0)
+    (property "MP" "C0603C105K4RACTU" (at 281.686 55.626 0)
       (effects (font (size 1.27 1.27)) hide)
     )
